File: PCB/Hyperion.kicad_pcb (KiCad board)
At the start: 2 copper layers, 118 parts, among them SW1 SW_PUSH, SW10 SW_PUSH, SW11 SW_PUSH, SW12 SW_PUSH, SW13 SW_PUSH, SW14 SW_PUSH, SW15 SW_PUSH, SW16 SW_PUSH, SW17 SW_PUSH, SW18 SW_PUSH, SW19 SW_PUSH, SW2 SW_PUSH, SW20 SW_PUSH, SW21 SW_PUSH, SW22 SW_PUSH, SW23 SW_PUSH, SW24 SW_PUSH, SW25 SW_PUSH, SW26 SW_PUSH, SW27 SW_PUSH, SW28 SW_PUSH, SW29 SW_PUSH, SW3 SW_PUSH, SW30 SW_PUSH, SW31 SW_PUSH, SW32 SW_PUSH, SW33 SW_PUSH, SW34 SW_PUSH, SW35 SW_PUSH, SW36 SW_PUSH, SW37 SW_PUSH, SW38 SW_PUSH, SW39 SW_PUSH, SW4 SW_PUSH, SW40 SW_PUSH, SW41 SW_PUSH, SW42 SW_PUSH, SW43 SW_PUSH, SW44 SW_PUSH, SW45 SW_PUSH, SW46 SW_PUSH, SW47 SW_PUSH, SW48 SW_PUSH, SW49 SW_PUSH, SW5 SW_PUSH, SW50 SW_PUSH, SW51 SW_PUSH, SW52 SW_PUSH, SW53 SW_PUSH, SW54 SW_PUSH, SW55 SW_PUSH, SW56 SW_PUSH, SW57 SW_PUSH, SW58 SW_PUSH, SW59 SW_PUSH, SW6 SW_PUSH, SW7 SW_PUSH, SW8 SW_PUSH, SW9 SW_PUSH, U1 ProMicro

Commit message: outlined
Parts:
- moved SW32 2.85 mm to (249.6, 178.9)
- moved U1 2.10 mm to (214.7, 96.4)
- moved SW34 0.11 mm to (259.2, 118.6)
- moved SW35 0.11 mm to (260.9, 137.6)
- moved SW36 0.11 mm to (262.6, 156.6)
- moved SW40 0.11 mm to (279.5, 131.2)
- moved SW52 0.11 mm to (335.4, 114.9)
- moved SW28 0.11 mm to (238.6, 101.3)
- moved SW29 0.11 mm to (240.3, 120.3)
- moved SW33 0.11 mm to (257.6, 99.7)
- moved SW38 0.11 mm to (276.1, 93.3)
- moved SW39 0.11 mm to (277.8, 112.2)
- moved SW42 0.11 mm to (295.4, 94.5)
- moved SW43 0.11 mm to (297.0, 113.1)
- moved SW51 0.11 mm to (333.7, 95.9)
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Other:
- board outline added: 309.6 x 123.8 mm
Changed lines of the file:
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@@
   (general
     (thickness 1.6)
-    (drawings 0)
+    (drawings 11)
     (tracks 0)
     (zones 0)
@@
     (solder_mask_min_width 0.25)
     (aux_axis_origin 0 0)
-    (visible_elements FFFFF77F)
+    (visible_elements 7FFFF7FF)
     (pcbplotparams
       (layerselection 0x010fc_ffffffff)
@@
   )
   (module emptystring:CherryMX_Hotswap_Back (layer F.Cu)
-    (at 238.598262 101.221366 5)
+    (at 238.598262 101.332054 5)
     (fp_text reference SW28 (at 7.1 8.2 5) (layer F.SilkS) hide
       (effects (font (size 1 1) (thickness 0.15)))
@@
   )
   (module emptystring:CherryMX_Hotswap_Back (layer F.Cu)
-    (at 240.258579 120.198875 5)
+    (at 240.258579 120.309563 5)
     (fp_text reference SW29 (at 7.1 8.2 5) (layer F.SilkS) hide
       (effects (font (size 1 1) (thickness 0.15)))
@@
   )
   (module emptystring:CherryMX_Hotswap_Back (layer F.Cu)
-    (at 241.918896 139.176384 5)
+    (at 241.918896 139.287072 5)
     (fp_text reference SW30 (at 7.1 8.2 5) (layer F.SilkS) hide
       (effects (font (size 1 1) (thickness 0.15)))
@@
   )
   (module emptystring:CherryMX_Hotswap_Back (layer F.Cu)
-    (at 243.579213 158.153893 5)
+    (at 243.579213 158.264581 5)
     (fp_text reference SW31 (at 7.1 8.2 5) (layer F.SilkS) hide
       (effects (font (size 1 1) (thickness 0.15)))
@@
   )
   (module emptystring:CherryMX_Hotswap_Back (layer F.Cu)
-    (at 246.770687 179.221481 10)
+    (at 249.6034 178.945728 10)
     (fp_text reference SW32 (at 7.1 8.2 10) (layer F.SilkS) hide
       (effects (font (size 1 1) (thickness 0.15)))
@@
   )
   (module emptystring:CherryMX_Hotswap_Back (layer F.Cu)
-    (at 257.575771 99.561049 5)
+    (at 257.575771 99.671737 5)
     (fp_text reference SW33 (at 7.1 8.2 5) (layer F.SilkS) hide
       (effects (font (size 1 1) (thickness 0.15)))
@@
   )
   (module emptystring:CherryMX_Hotswap_Back (layer F.Cu)
-    (at 259.236088 118.538558 5)
+    (at 259.236088 118.649246 5)
     (fp_text reference SW34 (at 7.1 8.2 5) (layer F.SilkS) hide
       (effects (font (size 1 1) (thickness 0.15)))
@@
   )
   (module emptystring:CherryMX_Hotswap_Back (layer F.Cu)
-    (at 260.896405 137.516067 5)
+    (at 260.896405 137.626755 5)
     (fp_text reference SW35 (at 7.1 8.2 5) (layer F.SilkS) hide
       (effects (font (size 1 1) (thickness 0.15)))
@@
   )
   (module emptystring:CherryMX_Hotswap_Back (layer F.Cu)
-    (at 262.556722 156.493576 5)
+    (at 262.556722 156.604264 5)
     (fp_text reference SW36 (at 7.1 8.2 5) (layer F.SilkS) hide
       (effects (font (size 1 1) (thickness 0.15)))
@@
   )
   (module emptystring:CherryMX_Hotswap_Back (layer F.Cu)
-    (at 273.705794 174.640927 5)
+    (at 273.705794 174.751614 5)
     (fp_text reference SW37 (at 7.1 8.2 5) (layer F.SilkS) hide
       (effects (font (size 1 1) (thickness 0.15)))
@@
   )
   (module emptystring:CherryMX_Hotswap_Back (layer F.Cu)
-    (at 276.138201 93.156355 5)
+    (at 276.138201 93.267043 5)
     (fp_text reference SW38 (at 7.1 8.2 5) (layer F.SilkS) hide
       (effects (font (size 1 1) (thickness 0.15)))
@@
   )
   (module emptystring:CherryMX_Hotswap_Back (layer F.Cu)
-    (at 277.798518 112.133864 5)
+    (at 277.798518 112.244552 5)
     (fp_text reference SW39 (at 7.1 8.2 5) (layer F.SilkS) hide
       (effects (font (size 1 1) (thickness 0.15)))
@@
   )
   (module emptystring:CherryMX_Hotswap_Back (layer F.Cu)
-    (at 279.458835 131.111373 5)
+    (at 279.458835 131.222061 5)
     (fp_text reference SW40 (at 7.1 8.2 5) (layer F.SilkS) hide
       (effects (font (size 1 1) (thickness 0.15)))
@@
   )
   (module emptystring:CherryMX_Hotswap_Back (layer F.Cu)
-    (at 281.119152 150.088882 5)
+    (at 281.119152 150.19957 5)
     (fp_text reference SW41 (at 7.1 8.2 5) (layer F.SilkS) hide
       (effects (font (size 1 1) (thickness 0.15)))
@@
   )
   (module emptystring:CherryMX_Hotswap_Back (layer F.Cu)
-    (at 295.364758 94.342664 5)
+    (at 295.364758 94.453352 5)
     (fp_text reference SW42 (at 7.1 8.2 5) (layer F.SilkS) hide
       (effects (font (size 1 1) (thickness 0.15)))
@@
   )
   (module emptystring:CherryMX_Hotswap_Back (layer F.Cu)
-    (at 296.991868 112.940623 5)
+    (at 296.991868 113.051311 5)
     (fp_text reference SW43 (at 7.1 8.2 5) (layer F.SilkS) hide
       (effects (font (size 1 1) (thickness 0.15)))
@@
   )
   (module emptystring:CherryMX_Hotswap_Back (layer F.Cu)
-    (at 298.652185 131.918132 5)
+    (at 298.652185 132.02882 5)
     (fp_text reference SW44 (at 7.1 8.2 5) (layer F.SilkS) hide
       (effects (font (size 1 1) (thickness 0.15)))
@@
   )
   (module emptystring:CherryMX_Hotswap_Back (layer F.Cu)
-    (at 300.312502 150.895641 5)
+    (at 300.312502 151.006329 5)
     (fp_text reference SW45 (at 7.1 8.2 5) (layer F.SilkS) hide
       (effects (font (size 1 1) (thickness 0.15)))
@@
   )
   (module emptystring:CherryMX_Hotswap_Back (layer F.Cu)
-    (at 314.757346 97.426725 5)
+    (at 314.757346 97.537412 5)
     (fp_text reference SW46 (at 7.1 8.2 5) (layer F.SilkS) hide
       (effects (font (size 1 1) (thickness 0.15)))
@@
   )
   (module emptystring:CherryMX_Hotswap_Back (layer F.Cu)
-    (at 316.417663 116.404234 5)
+    (at 316.417663 116.514921 5)
     (fp_text reference SW47 (at 7.1 8.2 5) (layer F.SilkS) hide
       (effects (font (size 1 1) (thickness 0.15)))
@@
   )
   (module emptystring:CherryMX_Hotswap_Back (layer F.Cu)
-    (at 318.07798 135.381743 5)
+    (at 318.07798 135.49243 5)
     (fp_text reference SW48 (at 7.1 8.2 5) (layer F.SilkS) hide
       (effects (font (size 1 1) (thickness 0.15)))
@@
   )
   (module emptystring:CherryMX_Hotswap_Back (layer F.Cu)
-    (at 319.738297 154.359252 5)
+    (at 319.738297 154.469939 5)
     (fp_text reference SW49 (at 7.1 8.2 5) (layer F.SilkS) hide
       (effects (font (size 1 1) (thickness 0.15)))
@@
   )
   (module emptystring:CherryMX_Hotswap_Back (layer F.Cu)
-    (at 333.734855 95.766408 5)
+    (at 333.734855 95.877096 5)
     (fp_text reference SW51 (at 7.1 8.2 5) (layer F.SilkS) hide
       (effects (font (size 1 1) (thickness 0.15)))
@@
   )
   (module emptystring:CherryMX_Hotswap_Back (layer F.Cu)
-    (at 335.395172 114.743917 5)
+    (at 335.395172 114.854605 5)
     (fp_text reference SW52 (at 7.1 8.2 5) (layer F.SilkS) hide
       (effects (font (size 1 1) (thickness 0.15)))
@@
   )
   (module emptystring:CherryMX_Hotswap_Back (layer F.Cu)
-    (at 337.055489 133.721426 5)
+    (at 337.055489 133.832114 5)
     (fp_text reference SW53 (at 7.1 8.2 5) (layer F.SilkS) hide
       (effects (font (size 1 1) (thickness 0.15)))
@@
   )
   (module emptystring:ProMicro_v2_Backside (layer F.Cu)
-    (at 214.73322 98.53651)
+    (at 214.73322 96.44103)
     (fp_text reference U1 (at -1.27 2.762 270) (layer F.SilkS) hide
       (effects (font (size 1 1) (thickness 0.15)))
@@
       (net 80 "Net-(U1-Pad24)"))
   )
+  (gr_line (start 379.81097 78.58158) (end 72.62843 78.58158) (layer Edge.Cuts) (width 0.12))
+  (gr_line (start 381.0016 189.31017) (end 381.0016 79.77221) (layer Edge.Cuts) (width 0.12))
+  (gr_line (start 379.81097 190.5008) (end 284.56057 190.5008) (layer Edge.Cuts) (width 0.12))
+  (gr_line (start 144.06623 190.5008) (end 72.62843 190.5008) (layer Edge.Cuts) (width 0.12))
+  (gr_line (start 71.4378 79.77221) (end 71.4378 189.31017) (layer Edge.Cuts) (width 0.12))
+  (gr_arc (start 72.62843 79.77221) (end 72.62843 78.58158) (angle -90) (layer Edge.Cuts) (width 0.12))
+  (gr_arc (start 72.62843 189.31017) (end 71.4378 189.31017) (angle -90) (layer Edge.Cuts) (width 0.12))
+  (gr_arc (start 379.81097 189.31017) (end 379.81097 190.5008) (angle -90) (layer Edge.Cuts) (width 0.12))
+  (gr_arc (start 379.81097 79.77221) (end 381.0016 79.77221) (angle -90) (layer Edge.Cuts) (width 0.12))
+  (gr_line (start 214.3134 202.4071) (end 144.06623 190.5008) (layer Edge.Cuts) (width 0.12))
+  (gr_line (start 284.56057 190.5008) (end 214.3134 202.4071) (layer Edge.Cuts) (width 0.12))
 )
